File: Hardware/TT7N v1.2.brd (EAGLE design)
At the start: 23 x 50 mm, 59 parts, among them U1 SPV1040, U3 XC6119

Commit message: Add files via upload
Parts:
- C14, C15, C16, C24: value 100n -> 100nF
- C22: value 10n -> 10nF
- C23: value 2.2n -> 2.2nF
- C3, C4: value 18p -> 18pF
- C5, C6: value 180p -> 180pF
- L2: value 53n -> 53nH
- L3: value 560n -> 560nH
- renumbered U$1 to U4, U$2 to U5, U$3 to U2, U$5 to U6, U$6 to U7
