File: Hardware/TT7N v1.2.sch (EAGLE design)
At the start: 59 parts, among them U1 SPV1040, U3 XC6119

Commit message: Add files via upload
Parts:
- renumbered U$1 to U4, U$2 to U5, U$3 to U2, U$5 to U6, U$6 to U7

Commit message: Add files via upload
Parts:
- C14, C15, C16, C24: value 100n -> 100nF
- C22: value 10n -> 10nF
- C23: value 2.2n -> 2.2nF
- C3, C4: value 18p -> 18pF
- C5, C6: value 180p -> 180pF
- L2: value 53n -> 53nH
- L3: value 560n -> 560nH
Changed lines of the file:
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@@
 <part name="U1" library="TT7" deviceset="SPV1040" device=""/>
 <part name="L1" library="TT7" deviceset="IND0402" device="" value=""/>
-<part name="L2" library="TT7" deviceset="IND0402" device="" value="53n"/>
+<part name="L2" library="TT7" deviceset="IND0402" device="" value="53nH"/>
 <part name="C1" library="TT7" deviceset="CAP0402" device="" value=""/>
 <part name="C2" library="TT7" deviceset="CAP0402" device="" value=""/>
-<part name="C3" library="TT7" deviceset="CAP0402" device="" value="18p"/>
-<part name="C4" library="TT7" deviceset="CAP0402" device="" value="18p"/>
+<part name="C3" library="TT7" deviceset="CAP0402" device="" value="18pF"/>
+<part name="C4" library="TT7" deviceset="CAP0402" device="" value="18pF"/>
 <part name="R1" library="TT7" deviceset="RES0402" device="" value="1M"/>
 <part name="R2" library="TT7" deviceset="RES0402" device="" value="1M"/>
-<part name="L3" library="TT7" deviceset="IND0402" device="" value="560n"/>
-<part name="C5" library="TT7" deviceset="CAP0402" device="" value="180p"/>
-<part name="C6" library="TT7" deviceset="CAP0402" device="" value="180p"/>
+<part name="L3" library="TT7" deviceset="IND0402" device="" value="560nH"/>
+<part name="C5" library="TT7" deviceset="CAP0402" device="" value="180pF"/>
+<part name="C6" library="TT7" deviceset="CAP0402" device="" value="180pF"/>
 <part name="LED1" library="TT7" deviceset="LED0603" device=""/>
 <part name="R5" library="TT7" deviceset="RES0402" device="" value="190R"/>
@@
 <part name="SUPPLY5" library="supply2" deviceset="GND" device=""/>
 <part name="R9" library="TT7" deviceset="RES0402" device="" value="1k"/>
-<part name="C14" library="TT7" deviceset="CAP0402" device="" value="100n"/>
-<part name="C15" library="TT7" deviceset="CAP0402" device="" value="100n"/>
+<part name="C14" library="TT7" deviceset="CAP0402" device="" value="100nF"/>
+<part name="C15" library="TT7" deviceset="CAP0402" device="" value="100nF"/>
 <part name="SUPPLY6" library="supply2" deviceset="GND" device=""/>
 <part name="SUPPLY7" library="supply2" deviceset="GND" device=""/>
@@
 <part name="SUPPLY9" library="supply2" deviceset="GND" device=""/>
 <part name="TCXO1" library="TT7" deviceset="TG2016SBN" device=""/>
-<part name="C16" library="TT7" deviceset="CAP0402" device="" value="100n"/>
+<part name="C16" library="TT7" deviceset="CAP0402" device="" value="100nF"/>
 <part name="SUPPLY10" library="supply2" deviceset="GND" device=""/>
 <part name="SUPPLY11" library="supply2" deviceset="GND" device=""/>
@@
 <part name="SUPPLY19" library="supply2" deviceset="GND" device=""/>
 <part name="SUPPLY20" library="supply2" deviceset="GND" device=""/>
-<part name="C22" library="TT7" deviceset="CAP0402" device="" value="10n"/>
-<part name="C23" library="TT7" deviceset="CAP0402" device="" value="2.2n"/>
-<part name="C24" library="TT7" deviceset="CAP0402" device="" value="100n"/>
+<part name="C22" library="TT7" deviceset="CAP0402" device="" value="10nF"/>
+<part name="C23" library="TT7" deviceset="CAP0402" device="" value="2.2nF"/>
+<part name="C24" library="TT7" deviceset="CAP0402" device="" value="100nF"/>
 <part name="SUPPLY21" library="supply2" deviceset="GND" device=""/>
 <part name="SUPPLY22" library="supply2" deviceset="GND" device=""/>
